Commit message: feat(mujoco): integrate real Mark7 model into generated URDF
Build the MuJoCo robot model by transforming Mark7 xacro and mounting it to Indy7 link6, with mesh path normalization and source path fallback.

Made-with: Cursor

File: mujoco_env/generated/indy7_mujoco.urdf (robot description, URDF)
Before this commit: robot indy, 9 links, 8 joints
Links:
- added link mark7_base_link, mass 0.35; collision mesh filename=mark7/base_link.stl scale=0.001 0.001 0.001; visual mesh filename=mark7/base_link.stl scale=0.001 0.001 0.001
- added link mark7_index_bottom_1, mass 0.04; collision mesh filename=mark7/index_bottom_1.stl scale=0.001 0.001 0.001; visual mesh filename=mark7/index_bottom_1.stl scale=0.001 0.001 0.001
- added link mark7_index_top_1, mass 0.03; collision mesh filename=mark7/index_top_1.stl scale=0.001 0.001 0.001; visual mesh filename=mark7/index_top_1.stl scale=0.001 0.001 0.001
- added link mark7_middle_bottom_1, mass 0.05; collision mesh filename=mark7/middle_bottom_1.stl scale=0.001 0.001 0.001; visual mesh filename=mark7/middle_bottom_1.stl scale=0.001 0.001 0.001
- added link mark7_middle_top_1, mass 0.03; collision mesh filename=mark7/middle_top_1.stl scale=0.001 0.001 0.001; visual mesh filename=mark7/middle_top_1.stl scale=0.001 0.001 0.001
- added link mark7_pinky_bottom_1, mass 0.03; collision mesh filename=mark7/pinky_bottom_1.stl scale=0.001 0.001 0.001; visual mesh filename=mark7/pinky_bottom_1.stl scale=0.001 0.001 0.001
- added link mark7_pinky_top_1, mass 0.03; collision mesh filename=mark7/pinky_top_1.stl scale=0.001 0.001 0.001; visual mesh filename=mark7/pinky_top_1.stl scale=0.001 0.001 0.001
- added link mark7_ringer_bottom_1, mass 0.04; collision mesh filename=mark7/ringer_bottom_1.stl scale=0.001 0.001 0.001; visual mesh filename=mark7/ringer_bottom_1.stl scale=0.001 0.001 0.001
- added link mark7_ringer_top_1, mass 0.03; collision mesh filename=mark7/ringer_top_1.stl scale=0.001 0.001 0.001; visual mesh filename=mark7/ringer_top_1.stl scale=0.001 0.001 0.001
- added link mark7_thumb_bottom_1, mass 0.05; collision mesh filename=mark7/thumb_bottom_1.stl scale=0.001 0.001 0.001; visual mesh filename=mark7/thumb_bottom_1.stl scale=0.001 0.001 0.001
- added link mark7_thumb_middle_1, mass 0.04; collision mesh filename=mark7/thumb_middle_1.stl scale=0.001 0.001 0.001; visual mesh filename=mark7/thumb_middle_1.stl scale=0.001 0.001 0.001
- added link mark7_thumb_top_1, mass 0.05; collision mesh filename=mark7/thumb_top_1.stl scale=0.001 0.001 0.001; visual mesh filename=mark7/thumb_top_1.stl scale=0.001 0.001 0.001
- link link0: geometry collision mesh filename=indy7/Indy7_0.stl; visual mesh filename=indy7/Indy7_0.stl
- link link1: geometry collision mesh filename=indy7/Indy7_1.stl; visual mesh filename=indy7/Indy7_1.stl
- link link2: geometry collision mesh filename=indy7/Indy7_2.stl; visual mesh filename=indy7/Indy7_2.stl
- link link3: geometry collision mesh filename=indy7/Indy7_3.stl; visual mesh filename=indy7/Indy7_3.stl
- link link4: geometry collision mesh filename=indy7/Indy7_4.stl; visual mesh filename=indy7/Indy7_4.stl
- link link5: geometry collision mesh filename=indy7/Indy7_5.stl; visual mesh filename=indy7/Indy7_5.stl
- link link6: geometry collision mesh filename=indy7/Indy7_6.stl; visual mesh filename=indy7/Indy7_6.stl
Joints:
- added joint mark7_base_index: type revolute, parent mark7_base_link, child mark7_index_bottom_1, origin xyz=-0.030299 -0.008352 0.089777 rpy=0 0 0, axis -0.997898 0.03262 -0.055994, limit lower=0.0 upper=1.396 effort=20 velocity=2.0
- added joint mark7_base_middle: type revolute, parent mark7_base_link, child mark7_middle_bottom_1, origin xyz=-0.008513 -0.011057 0.092109 rpy=0 0 0, axis -0.998722 0.009815 0.049588, limit lower=0.0 upper=1.396 effort=20 velocity=2.0
- added joint mark7_base_pinky: type revolute, parent mark7_base_link, child mark7_pinky_bottom_1, origin xyz=0.031928 -0.005928 0.078169 rpy=0 0 0, axis -0.972127 -0.033995 0.231975, limit lower=0.0 upper=1.396 effort=20 velocity=2.0
- added joint mark7_base_ringer: type revolute, parent mark7_base_link, child mark7_ringer_bottom_1, origin xyz=0.011471 -0.009409 0.085649 rpy=0 0 0, axis -0.991562 -0.005724 0.129511, limit lower=0.0 upper=1.396 effort=20 velocity=2.0
- added joint mark7_base_thumb: type revolute, parent mark7_base_link, child mark7_thumb_bottom_1, origin xyz=-0.007376 0.005575 0.034463 rpy=0 0 0, axis -0.995619 0.092558 -0.013228, limit lower=0.0 upper=1.396 effort=25 velocity=2.0
- added joint mark7_index_bottom_top_rev: type revolute, parent mark7_index_bottom_1, child mark7_index_top_1, origin xyz=-0.002315 0.007076 0.037929 rpy=0 0 0, axis -0.997898 0.03262 -0.055994, limit lower=0.0 upper=1.396 effort=0 velocity=4.0, mimic joint=mark7_base_index multiplier=1.0 offset=0
- added joint mark7_middle_bottom_top_rev: type revolute, parent mark7_middle_bottom_1, child mark7_middle_top_1, origin xyz=0.001564 0.008692 0.041538 rpy=0 0 0, axis -0.998722 0.009815 0.049588, limit lower=0.0 upper=1.396 effort=0 velocity=4.0, mimic joint=mark7_base_middle multiplier=1.0 offset=0
- added joint mark7_mount_joint: type fixed, parent link6, child mark7_base_link, origin xyz=0.000 0.000 0.085 rpy=0 0 0
- added joint mark7_pinky_bottom_top: type revolute, parent mark7_pinky_bottom_1, child mark7_pinky_top_1, origin xyz=0.005511 0.006642 0.029486 rpy=0 0 0, axis -0.972127 -0.033995 0.231975, limit lower=0.0 upper=1.396 effort=0 velocity=2.0, mimic joint=mark7_base_pinky multiplier=1.0 offset=0
- added joint mark7_ringer_bottom_top_rev: type revolute, parent mark7_ringer_bottom_1, child mark7_ringer_top_1, origin xyz=0.004246 0.008569 0.037454 rpy=0 0 0, axis -0.991562 -0.005724 0.129511, limit lower=0.0 upper=1.396 effort=0 velocity=4.0, mimic joint=mark7_base_ringer multiplier=1.0 offset=0
- added joint mark7_thumb_bottom_middle_rev: type revolute, parent mark7_thumb_bottom_1, child mark7_thumb_middle_1, origin xyz=-0.029041 0.009347 -0.000505 rpy=0 0 0, axis -0.092166 -0.947763 0.305369, limit lower=-0.872665 upper=0.0 effort=30 velocity=2.0
- added joint mark7_thumb_middle_top_rev: type revolute, parent mark7_thumb_middle_1, child mark7_thumb_top_1, origin xyz=-0.022653 0.00116 0.007686 rpy=0 0 0, axis -0.092165 -0.947763 0.305369, limit lower=-0.872665 upper=0.0 effort=0 velocity=2.0, mimic joint=mark7_thumb_bottom_middle_rev multiplier=1.0 offset=0
